Commit message: exp0.2 Phase2 参考轨迹行走：mocap 全身查表(2b) + 逐段周期 + URDF 右臂限位修复 + ref_lib 入库
- prep_mocap_ref.py: GMR→ref_lib.pt（Isaac序重排/翻转/120→50Hz/自相关周期/锚点/整周期切段/限位clip）
- env: _init_mocap_lib 加载器 + _current_seg_id 指令分档 + _get_phase 逐段周期 + compute_ref_state 查表（mocap_full_body 全身）
- 修复周期帧数单位错位（P=114→57，按库 fps 而非 policy dt）
- config: use_mocap_ref/mocap_full_body=True, ref_joint_pos 1.8, 右臂 default 镜像取反
- URDF: right_shoulder_roll[-2,0]→[0,2], right_elbow_pitch[0,2]→[-2,0]
- test_mocap_ref_lookup.py 6 项单测 + ref_lib.pt 强制入库（绕过 *.pt 忽略）

File: resources/robots/x1/urdf/X1_29DOF_physically_mirrored.urdf (robot description, URDF)
Before this commit: robot x1, 60 links, 59 joints
Joints:
- joint right_elbow_pitch_joint: limit lower=0.0 upper=2.0 effort=20.0 velocity=13.61 -> lower=-2.0 upper=0.0 effort=20.0 velocity=13.61
- joint right_shoulder_roll_joint: limit lower=-2 upper=0 effort=20.0 velocity=13.61 -> lower=0 upper=2 effort=20.0 velocity=13.61

Commit message: exp2.3 前置：URDF 右臂/右踝 6 关节轴对齐真机约定（修真机反向）
真机症状：right_ankle_pitch / right_elbow_pitch 等关节在真机上反向。
根因：训练 URDF 的世界轴方向与真机重定向模型 czy/diff/gmr_x1_assets/x1.xml
相反；该模型与 sim2sim 模型 xyber_x1_serial.xml 一致，且与 prep_mocap_ref.py
的 FLIP_JOINTS 6 关节集合逐字相同 —— 此前只修了数据侧（FLIP_JOINTS），
URDF/部署侧未修，故真机反向。

改动（4 文件 + ref_lib）：
- URDF：shoulder p/r/y、elbow p/y、ankle pitch 轴翻正（axis/range 对齐 gmr）；
  还原 4 处无依据的 wrist 轴改动
- MJCF x1_29dof_raw.xml：同步翻同 6 关节（prep 的 FK 校验依赖它）
- prep_mocap_ref.py：FLIP_JOINTS 清空（URDF 已与真机同约定）
- config：6 关节 default 取反 + swing[10] 取反；更新依赖旧约定的注释
- ref_lib.pt：重导 4 段（972/965/683/120）

验证：世界轴 29/29 对齐 gmr、12/12 对齐 sim2sim；默认位姿物理形状逐位保持
（59 link 最大偏差 0.00000m）；prep FK 校验 0.3mm/6.05mm 通过。

影响：本次为坐标重标定（sim 物理与改前同构），但旧 checkpoint 语义过期 →
exp2.3 必须从头训练，不可续训。

File: resources/robots/x1/urdf/X1_29DOF_physically_mirrored.urdf (robot description, URDF)
Before this commit: robot x1, 60 links, 59 joints
Joints:
- joint right_ankle_pitch_joint: axis 0 0 -1 -> 0 0 1
- joint right_elbow_pitch_joint: axis 0 0 1 -> 0 0 -1; limit lower=-2.0 upper=0.0 effort=20.0 velocity=13.61 -> lower=0.0 upper=2.0 effort=20.0 velocity=13.61
- joint right_elbow_yaw_joint: axis 0 0 1 -> 0 0 -1
- joint right_shoulder_pitch_joint: axis 0 0 -1 -> 0 0 1
- joint right_shoulder_roll_joint: axis 0 0 -1 -> 0 0 1; limit lower=0 upper=2 effort=20.0 velocity=13.61 -> lower=-2 upper=0 effort=20.0 velocity=13.61
- joint right_shoulder_yaw_joint: axis 0 0 -1 -> 0 0 1
